File: gampad.kicad_sch (KiCad schematic)
At the start: 26 parts, among them J1 swd header, J10 Conn_01x01, J3 Conn_01x01, J4 Conn_01x01, J5 Conn_01x01, J6 Conn_01x01, J7 Conn_01x01, J8 Conn_01x01, J9 Conn_01x01, U1 STM32L442KCUx, U2 MIC5504-3.3YM5

Commit message: heheh
Changed lines of the file:
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@@
 		(fields_autoplaced yes)
 		(property "Reference" "U1"
-			(at 209.9467 76.2 0)
+			(at 215.2081 73.66 0)
 			(show_name no)
 			(do_not_autoplace no)
@@
 					(size 1.27 1.27)
 				)
-				(justify left)
+				(justify right)
 			)
 		)
 		(property "Value" "STM32L442KCUx"
-			(at 209.9467 73.66 0)
+			(at 215.2081 76.2 0)
 			(show_name no)
 			(do_not_autoplace no)
@@
 					(size 1.27 1.27)
 				)
-				(justify left)
+				(justify right)
 			)
 		)
