File: sch+pcb/_restore_backup_2026-09-13T20-50-06-499/gampad.kicad_pcb (KiCad board)
At the start: 2 copper layers, 85.6 x 53.4 mm, 43 parts, among them J1 swd header, J10 Conn_01x01, J3 Conn_01x01, J4 Conn_01x01, J5 Conn_01x01, J6 Conn_01x01, J7 Conn_01x01, J8 Conn_01x01, J9 Conn_01x01, U1 STM32L442KCUx, U2 MIC5504-3.3YM5

Commit message: woah stuff goshhhhh
Parts:
- moved G*** 0.72 mm to (105.0, 93.8)
- moved G*** 0.35 mm to (105.8, 93.6)
